File: Kicad Files/Lisa_Floppy_Power.kicad_pcb (KiCad board)
At the start: 2 copper layers, 198.1 x 50.8 mm, 35 parts, among them J1 Lisa KB In, J10 PWR_SW, J11 Audio_Video, J14 Speaker Out, J15 Arduino_Pro_Micro_5V_16MHz, J16 Lisa_Floppy, J17 Sony Floppy Connector, J2 +5V, J3 +12V, J4 ATX-24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

Commit message: Add files via upload
KiCad files with updated 7905 footprint
Parts:
- moved U1 5.07 mm to (182.1, 46.0), turned to 90 degrees
Connections:
- U1 pad 1: GND-R -> -5V_7905
- U1 pad 3: -5V_7905 -> GND-R
Other:
- board text added: "Out"
